Commit message: Update rosbotxl urdf

File: robot_models/rosbotxl/rosbot_xl.urdf (robot description, URDF)
Before this commit: robot rosbot_xl, 9 links, 8 joints
Links:
- removed link front_left_wheel_link
- removed link front_right_wheel_link
- removed link imu
- removed link rear_left_wheel_link
- removed link rear_right_wheel_link
- added link fl_wheel_link, mass 0.051; collision cylinder length=0.032 radius=0.048; visual mesh filename=file:///robot_models/rosbotxl/meshes/wheel_a.dae scale=1 1 1
- added link fr_wheel_link, mass 0.051; collision cylinder length=0.032 radius=0.048; visual mesh filename=file:///robot_models/rosbotxl/meshes/wheel_b.dae scale=1 1 1
- added link imu_link, mass 0.0000001
- added link rl_wheel_link, mass 0.051; collision cylinder length=0.032 radius=0.048; visual mesh filename=file:///robot_models/rosbotxl/meshes/wheel_a.dae scale=1 1 1
- added link rplidar_s1_link, mass 0.105; collision cylinder length=0.051 radius=0.02775; visual mesh filename=file:///robot_models/rosbotxl/meshes/rplidar_s1.stl scale=0.0001 0.0001 0.0001
- added link rr_wheel_link, mass 0.051; collision cylinder length=0.032 radius=0.048; visual mesh filename=file:///robot_models/rosbotxl/meshes/wheel_b.dae scale=1 1 1
- link laser: mass 0.105 -> None; geometry 
Joints:
- removed joint base_link_to_body_joint
- removed joint body_link_to_imu_joint
- removed joint front_left_wheel_joint
- removed joint front_right_wheel_joint
- removed joint rear_left_wheel_joint
- removed joint rear_right_wheel_joint
- added joint base_to_body_joint: type fixed, parent base_link, child body_link, origin xyz=0.0 0.0 0.048 rpy=0.0 0.0 0.0
- added joint body_to_imu_joint: type fixed, parent body_link, child imu_link, origin xyz=-0.1369 -0.0419 0.0370 rpy=3.14159 0.0 0.0
- added joint cover_link_to_rplidar_s1_link_joint: type fixed, parent cover_link, child rplidar_s1_link, origin xyz=0.0 0.0 0.0 rpy=0.0 0.0 3.141592653589793
- added joint fl_wheel_joint: type continuous, parent body_link, child fl_wheel_link, origin xyz=0.085 0.118 0.0 rpy=0.0 0.0 0.0, axis 0.0 1.0 0.0, limit effort=1.2 velocity=21.0
- added joint fr_wheel_joint: type continuous, parent body_link, child fr_wheel_link, origin xyz=0.085 -0.118 0.0 rpy=0.0 0.0 0.0, axis 0.0 1.0 0.0, limit effort=1.2 velocity=21.0
- added joint rl_wheel_joint: type continuous, parent body_link, child rl_wheel_link, origin xyz=-0.085 0.118 0.0 rpy=0.0 0.0 0.0, axis 0.0 1.0 0.0, limit effort=1.2 velocity=21.0
- added joint rr_wheel_joint: type continuous, parent body_link, child rr_wheel_link, origin xyz=-0.085 -0.118 0.0 rpy=0.0 0.0 0.0, axis 0.0 1.0 0.0, limit effort=1.2 velocity=21.0
- joint laser_joint: origin xyz=0 0 0.04 rpy=0.0 0.0 0.0 -> xyz=0.0 0.0 0.04 rpy=0.0 0.0 0.0; parent cover_link -> rplidar_s1_link
