Commit message: Refactor rosbot2 description

File: robot_models/rosbot2/rosbot2.urdf (robot description, URDF)
Before this commit: robot rosbot, 14 links, 13 joints
Links:
- removed link camera_depth_frame
- removed link camera_rgb_frame
- removed link front_left_wheel
- removed link front_right_wheel
- removed link range_fl
- removed link range_fr
- removed link range_rl
- removed link range_rr
- removed link rear_left_wheel
- removed link rear_right_wheel
- removed link top
- added link body_link, mass 2.0; collision box size=0.197 0.150 0.080; visual mesh filename=file:///robot_models/rosbot2/meshes/body.stl scale=0.001 0.001 0.001
- added link cover_link, mass 0.000001; visual mesh filename=file:///robot_models/rosbot2/meshes/cover.stl scale=0.001 0.001 0.001
- added link fl_range
- added link fl_wheel_link, mass 0.100; collision cylinder length=0.036 radius=0.0425; visual mesh filename=file:///robot_models/rosbot2/meshes/wheel.stl scale=0.001 0.001 0.001
- added link fr_range
- added link fr_wheel_link, mass 0.100; collision cylinder length=0.036 radius=0.0425; visual mesh filename=file:///robot_models/rosbot2/meshes/wheel.stl scale=0.001 0.001 0.001
- added link imu_link, mass 0.001
- added link orbbec_astra_depth_link
- added link orbbec_astra_depth_reference_link
- added link orbbec_astra_link, mass 0.105; collision box size=0.165 0.04 0.05; visual mesh filename=file:///robot_models/rosbot2/meshes/astra.stl scale=0.001 0.001 0.001
- added link rl_range
- added link rl_wheel_link, mass 0.100; collision cylinder length=0.036 radius=0.0425; visual mesh filename=file:///robot_models/rosbot2/meshes/wheel.stl scale=0.001 0.001 0.001
- added link rplidar_a2_link, mass 0.190; collision cylinder length=0.0408 radius=0.03625; visual mesh filename=file:///robot_models/rosbot2/meshes/rplidar.stl scale=0.001 0.001 0.001
- added link rr_range
- added link rr_wheel_link, mass 0.100; collision cylinder length=0.036 radius=0.0425; visual mesh filename=file:///robot_models/rosbot2/meshes/wheel.stl scale=0.001 0.001 0.001
- link base_link: mass 5 -> None; geometry 
- link camera_link: mass 1e-5 -> 0.000001; geometry 
- link laser: mass 1e-5 -> None; geometry 
Joints:
- removed joint astra_joint
- removed joint camera_depth_joint
- removed joint camera_optical_joint
- removed joint front_left_wheel_hinge
- removed joint front_right_wheel_hinge
- removed joint range_fl_joint
- removed joint range_fr_joint
- removed joint range_rl_joint
- removed joint range_rr_joint
- removed joint rear_left_wheel_hinge
- removed joint rear_right_wheel_hinge
- removed joint rplidar_joint
- removed joint top_joint
- added joint base_to_body_joint: type fixed, parent base_link, child body_link, origin xyz=0.0 0.0 0.0425 rpy=0.0 0.0 0.0
- added joint body_to_camera_joint: type fixed, parent body_link, child camera_link, origin xyz=-0.0141 0.0 0.125 rpy=0.0 0.0 0.0
- added joint body_to_cover_joint: type fixed, parent body_link, child cover_link, origin xyz=0.0 0.0 0.060 rpy=0.0 0.0 0.0
- added joint body_to_imu_joint: type fixed, parent body_link, child imu_link, origin xyz=-0.1369 -0.0419 0.0370 rpy=0.0 0.0 0.0
- added joint body_to_orbbec_astra_joint: type fixed, parent camera_link, child orbbec_astra_link, origin xyz=0.0 0.0 0.0 rpy=0.0 0.0 0.0
- added joint cover_link_to_rplidar_a2_link_joint: type fixed, parent cover_link, child rplidar_a2_link, origin xyz=0.02 0.0 0.0 rpy=0.0 0.0 -3.141592653589793
- added joint fl_range_joint: type fixed, parent body_link, child fl_range, origin xyz=0.1 0.05 0.01 rpy=0 0 0.13 , axis 0 1 0
- added joint fl_wheel_joint: type continuous, parent body_link, child fl_wheel_link, origin xyz=0.053 0.096 0.0 rpy=0.0 0.0 0.0, axis 0.0 1.0 0.0, limit effort=1.5 velocity=5.0
- added joint fr_range_joint: type fixed, parent body_link, child fr_range, origin xyz=0.1 -0.05 0.01 rpy=0 0 -0.13 , axis 0 1 0
- added joint fr_wheel_joint: type continuous, parent body_link, child fr_wheel_link, origin xyz=0.053 -0.096 0.0 rpy=0.0 0.0 0.0, axis 0.0 1.0 0.0, limit effort=1.5 velocity=5.0
- added joint laser_joint: type fixed, parent rplidar_a2_link, child laser, origin xyz=0.0 0.0 0.0335 rpy=0.0 0.0 0.0
- added joint orbbec_astra_depth_joint: type fixed, parent orbbec_astra_link, child orbbec_astra_depth_link, origin xyz=0.01 0 0.035 rpy=0.0 1.5707963267948966 0.0
- added joint orbbec_astra_depth_reference_joint: type fixed, parent orbbec_astra_depth_link, child orbbec_astra_depth_reference_link, origin xyz=0.0 0.0 0.0 rpy=1.5707963267948966 -1.5707963267948966 0.0
- added joint rl_range_joint: type fixed, parent body_link, child rl_range, origin xyz=-0.1 0.05 0.01 rpy=0 0 3.01 , axis 0 1 0
- added joint rl_wheel_joint: type continuous, parent body_link, child rl_wheel_link, origin xyz=-0.053 0.096 0.0 rpy=0.0 0.0 0.0, axis 0.0 1.0 0.0, limit effort=1.5 velocity=5.0
- added joint rr_range_joint: type fixed, parent body_link, child rr_range, origin xyz=-0.1 -0.05 0.01 rpy=0 0 3.27 , axis 0 1 0
- added joint rr_wheel_joint: type continuous, parent body_link, child rr_wheel_link, origin xyz=-0.053 -0.096 0.0 rpy=0.0 0.0 0.0, axis 0.0 1.0 0.0, limit effort=1.5 velocity=5.0

Commit message: Fix transforms

File: robot_models/rosbot2/rosbot2.urdf (robot description, URDF)
Before this commit: robot rosbot, 18 links, 17 joints
Joints:
- joint body_to_cover_joint: origin xyz=0.0 0.0 0.060 rpy=0.0 0.0 0.0 -> xyz=0.0 0.0 0.0603 rpy=0.0 0.0 0.0
- joint body_to_imu_joint: origin xyz=-0.1369 -0.0419 0.0370 rpy=0.0 0.0 0.0 -> xyz=0.003 -0.0495 0.04332 rpy=0.0 0.0 0.0
- joint fl_range_joint: origin xyz=0.1 0.05 0.01 rpy=0 0 0.13  -> xyz=0.0926 0.05 0.015 rpy=0 0 0.218 
- joint fr_range_joint: origin xyz=0.1 -0.05 0.01 rpy=0 0 -0.13  -> xyz=0.0926 -0.05 0.015 rpy=0 0 -0.218 
- joint rl_range_joint: origin xyz=-0.1 0.05 0.01 rpy=0 0 3.01  -> xyz=-0.0926 0.05 0.0115 rpy=0 0 2.924 
- joint rr_range_joint: origin xyz=-0.1 -0.05 0.01 rpy=0 0 3.27  -> xyz=-0.0926 -0.05 0.0115 rpy=0 0 3.360
